File: Hardware/PCB_HORNO/PCB_HORNO.kicad_sch (KiCad schematic)
At the start: 86 parts, among them J1 Screw_Terminal_01x20, J2 Screw_Terminal_01x20, J3 Screw_Terminal_01x20, J4 Screw_Terminal_01x20

Commit message: Integrando todas las interfaces
Parts:
- added C3, C4, C5, C6: 10nF, Capacitor_THT:C_Disc_D4.3mm_W1.9mm_P5.00mm, symbol Device:C
- added D1, D2, D3, D4, D5, D6, D7, D8: LED, LED_THT:LED_D4.0mm, symbol Device:LED
- added J0_1, J0_2, J0_3, J0_4, J0_5, J0_6, J9_1, J9_2, J9_3, J9_4, J9_5, J9_6: Screw_Terminal_01x03, TerminalBlock_Phoenix:TerminalBlock_Phoenix_PT-1,5-3-3.5-H_1x03_P3.50mm_Horizontal, symbol Connector:Screw_Terminal_01x03
- added J1-1, J1-2, J1-3, J1-4, J2-1, J2-2, J2-3, J2-4, J3-1, J3-2, J3-3, J3-4, J4-1, J4-2, J4-3, J4-4, J5-1, J5-2, J5-3, J5-4, J6-1, J6-2, J6-3, J6-4, J7-1, J7-2, J7-3, J7-4, J8-1, J8-2, J8-3, J8-4: Screw_Terminal_01x01, TerminalBlock_MetzConnect:TerminalBlock_MetzConnect_360271_1x01_Horizontal_ScrewM3.0_Boxed, symbol Connector:Screw_Terminal_01x01
- added PX45, PX46, PX47, PX48, PX49, PX50, PX51, PX52, PX53, PX54, PX55, PX56, PX57, PX58, PX59, PX60, PX61, PX62, PX63, PX64, PX65, PX66, PX67, PX68, PX69, PX70, PX71, PX72, PX73, PX74, PX75, PX76, PX77, PX78, PX79, PX80, PX81, PX82, PX83, PX84, PX85, PX86, PX87, PX88, PX89, PX90, PX91, PX92: ~, Connector_Wire:SolderWire-0.75sqmm_1x01_D1.25mm_OD2.3mm, symbol Connector:Screw_Terminal_01x01
- added Q1, Q2, Q3, Q4: 2N2222, Package_TO_SOT_THT:TO-39-3, symbol Transistor_BJT:2N2219
- added R1, R2, R3, R4, R5, R6, R7, R8: 560 Ω 1/4 W, Resistor_THT:R_Axial_DIN0207_L6.3mm_D2.5mm_P10.16mm_Horizontal, symbol Device:R_US
- added U1, U2, U3, U4, U5, U6, U7, U8: TLP521-1, Package_DIP:DIP-4_W7.62mm, symbol Isolator:Optocoupler_DC_PhotoNPN_AKEC
- added U10, U11, U12, U9: LM741, LM741_TH:LM741_TH, symbol Amplifier_Operational:LM741
Connections:
- new net: D3.1 (K), U3.1
- new net: D3.2 (A), J3-2.1 (Pin_1)
- new net: D5.1 (K), U5.1
- new net: J0_1.1 (Pin_1), U1.2, U2.2, U3.2, U4.2, U5.2, U6.2, U7.2, U8.2
- new net: J9_3.3 (Pin_3), R5.1, U5.3
- new net: J9_1.3 (Pin_3), U1.4, U2.4, U3.4, U4.4, U5.4, U6.4, U7.4, U8.4
- new net: J0_3.2 (Pin_2), J7-1.1 (Pin_1)
- new net: J9_2.2 (Pin_2), R3.1, U3.3
- new net: J1-3.1 (Pin_1), U9.2 (-), U9.6
- new net: C6.1, J0_5.1 (Pin_1), U9.3 (+)
- new net: J0_4.2 (Pin_2), U10.4 (V-), U11.4 (V-), U12.4 (V-), U9.4 (V-)
- new net: J0_4.1 (Pin_1), U10.7 (V+), U11.7 (V+), U12.7 (V+), U9.7 (V+)
- new net: C4.1, J0_5.3 (Pin_3), U11.3 (+)
- new net: J0_2.1 (Pin_1), J3-1.1 (Pin_1)
- new net: J2-3.1 (Pin_1), U10.2 (-), U10.6
- new net: J3-3.1 (Pin_1), U11.2 (-), U11.6
- new net: J9_4.3 (Pin_3), R8.1, U8.3
- new net: J9_1.2 (Pin_2), R1.2, R2.2, R3.2, R4.2, R5.2, R6.2, R7.2, R8.2
- new net: C5.1, J0_5.2 (Pin_2), U10.3 (+)
- new net: D8.1 (K), U8.1
- new net: J0_1.2 (Pin_2), J1-1.1 (Pin_1)
- new net: J0_1.3 (Pin_3), J2-1.1 (Pin_1)
- new net: J4-4.1 (Pin_1), Q4.2 (B)
- new net: J9_3.1 (Pin_1), R7.1, U7.3
- new net: J9_3.2 (Pin_2), R6.1, U6.3
- new net: J0_3.1 (Pin_1), J6-1.1 (Pin_1)
- new net: J5-4.1 (Pin_1), Q1.1 (E)
- new net: C3.1, J0_6.1 (Pin_1), U12.3 (+)
- new net: J0_2.2 (Pin_2), J4-1.1 (Pin_1)
- new net: J0_2.3 (Pin_3), J5-1.1 (Pin_1)
- new net: J6-4.1 (Pin_1), Q2.1 (E)
- new net: J2-4.1 (Pin_1), Q2.2 (B)
- new net: Q1.3 (C), Q2.3 (C), Q3.3 (C), Q4.3 (C)
- new net: J1-4.1 (Pin_1), Q1.2 (B)
- new net: D4.2 (A), J4-2.1 (Pin_1)
- new net: D8.2 (A), J8-2.1 (Pin_1)
- new net: D2.1 (K), U2.1
- new net: D2.2 (A), J2-2.1 (Pin_1)
- new net: D1.1 (K), U1.1
- new net: D1.2 (A), J1-2.1 (Pin_1)
- new net: J0_3.3 (Pin_3), J8-1.1 (Pin_1)
- new net: D7.1 (K), U7.1
- new net: J9_2.1 (Pin_1), R4.1, U4.3
- new net: J9_2.3 (Pin_3), R2.1, U2.3
- new net: D5.2 (A), J5-2.1 (Pin_1)
- new net: J9_1.1 (Pin_1), R1.1, U1.3
- new net: J8-4.1 (Pin_1), Q4.1 (E)
- new net: D6.2 (A), J6-2.1 (Pin_1)
- new net: J4-3.1 (Pin_1), U12.2 (-), U12.6
- new net: D4.1 (K), U4.1
- new net: D6.1 (K), U6.1
- new net: D7.2 (A), J7-2.1 (Pin_1)
- new net: J7-4.1 (Pin_1), Q3.1 (E)
- new net: J3-4.1 (Pin_1), Q3.2 (B)
- new net GNDREF: C3.2, C4.2, C5.2, C6.2, J0_4.3 (Pin_3), J5-3.1 (Pin_1), J6-3.1 (Pin_1), J7-3.1 (Pin_1), J8-3.1 (Pin_1)
Other:
- moved on the sheet: 3V3a1, 3V3b1, 5Va1, 5Vb1, C1, C2, GND1, GND2, GND3, J1, J2, J3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

Commit message: Reorganizando elementos
Other:
- moved on the sheet: 3V3a1, 3V3b1, 5Va1, 5Vb1, C3, C4, C5, C6, D1, D2, D3, D4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

Commit message: Reorganizando elementos
Parts:
- removed J9_2, J9_3, J9_4, J9_6: Screw_Terminal_01x03, TerminalBlock_Phoenix:TerminalBlock_Phoenix_PT-1,5-3-3.5-H_1x03_P3.50mm_Horizontal, symbol Connector:Screw_Terminal_01x03
- added PX100, PX101, PX102, PX103, PX104, PX105, PX106, PX107, PX108, PX109, PX110, PX111, PX112, PX113, PX114, PX115, PX116, PX117, PX118, PX119, PX120, PX121, PX122, PX123, PX124, PX93, PX94, PX95, PX96, PX97, PX98, PX99: ~, Connector_Wire:SolderWire-0.75sqmm_1x01_D1.25mm_OD2.3mm, symbol Connector:Screw_Terminal_01x01
- U10, U11, U12, U9: footprint LM741_TH:LM741_TH -> LM741_TH:LM471_TH
Connections:
- net GNDREF: now also J0_4.1 (Pin_1), J9_5.3 (Pin_3); no longer J0_4.3 (Pin_3)
- net at U10.7 (V+), U11.7 (V+), U12.7 (V+)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: now also J0_4.3 (Pin_3); no longer J0_4.1 (Pin_1)
- net at R1.2, R2.2, R3.2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: now also J9_1.1 (Pin_1), R1.1, U1.3; no longer J9_1.2 (Pin_2)
- net at Q1.3 (C), Q2.3 (C), Q3.3 (C)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: now also J9_5.1 (Pin_1)
Other:
- moved on the sheet: C3, C4, C5, C6, D1, D2, D3, D4, D5, D6, D7, D8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

Commit message: Integración de nuevos modulos al PCB (puente H, detector de cruce por cero, disparo con triac, salida analogica amplificada)
Parts:
- added C7: 10nF, Capacitor_THT:C_Disc_D4.3mm_W1.9mm_P5.00mm, symbol Device:C
- added D9: D_Bridge_+-AA, symbol Device:D_Bridge_+-AA
- added J0_10, J0_11, J0_7, J0_8, J0_9: Screw_Terminal_01x03, TerminalBlock_Phoenix:TerminalBlock_Phoenix_PT-1,5-3-3.5-H_1x03_P3.50mm_Horizontal, symbol Connector:Screw_Terminal_01x03
- added Q5: BTA16-800B, Package_TO_SOT_THT:TO-220-3_Vertical, symbol Triac_Thyristor:BTA16-800B
- added Q6, Q7: Q_PNP, symbol Device:Q_PNP
- added Q8, Q9: Q_NPN, symbol Device:Q_NPN
- added R10, R11, R12, R13, R14, R15, R16, R17, R9: R_US, symbol Device:R_US
- added RV1, RV2, RV3: R_Potentiometer_US, symbol Device:R_Potentiometer_US
- added U13: MOC3021M, Package_DIP:DIP-6_W7.62mm, symbol Relay_SolidState:MOC3021M
- added U14: TLP521-1, Package_DIP:DIP-4_W7.62mm, symbol Isolator:Optocoupler_DC_PhotoNPN_AKEC
- added U15: 4069, symbol 4xxx:4069
- added U16: LM741, LM741_TH:LM471_TH, symbol Amplifier_Operational:LM741
Connections:
- net GNDREF: now also C7.2, RV3.1, U13.2
- new net: J0_8.1 (Pin_1), R9.1
- new net: D9.3, R9.2
- new net: Q7.B, R17.1
- new net: J0_10.3 (Pin_3), Q6.C, Q7.C
- new net: J0_9.3 (Pin_3), Q7.E, Q9.E
- new net: R12.1, U14.4
- new net: J0_11.3 (Pin_3), R12.2
- new net: J0_7.1 (Pin_1), Q5.1 (A1)
- new net: J0_7.3 (Pin_3), Q5.2 (A2), R13.2
- new net: Q6.B, R15.2
- new net: J0_9.1 (Pin_1), Q6.E, Q8.E
- new net: RV2.1, RV3.2, U16.2 (-)
- new net: C7.1, U16.3 (+)
- new net: R13.1, U13.6
- new net: R16.2, R17.2, U15.2
- new net: Q5.3 (G), U13.4
- new net: R14.1, R15.1, U15.1
- new net: Q8.B, R14.2
- new net: J0_8.3 (Pin_3), R10.1
- new net: R11.2, U14.1
- new net: D9.2 (-), U14.2
- new net: J0_11.1 (Pin_1), U14.3
- new net: D9.1 (+), R11.1
- new net: D9.4, R10.2
- new net: J0_10.1 (Pin_1), Q8.C, Q9.C
- new net: RV2.2, U16.6
- new net: Q9.B, R16.1
Other:
- note added: "ESP32"
- note added: "Entradas/Salidas"
- note added: "Otro ESP32 u otros modulos"
- moved on the sheet: C3, C4, C5, C6, D1, D2, D3, D4, D5, D6, D7, D8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

Commit message: Integrando nuevos modulos al PCB
Parts:
- removed J1-1, J1-2, J2-1, J2-2, J3-1, J3-2, J4-1, J4-2, J5-1, J5-2, J6-1, J6-2, J7-1, J7-2, J8-1, J8-2: Screw_Terminal_01x01, TerminalBlock_MetzConnect:TerminalBlock_MetzConnect_360271_1x01_Horizontal_ScrewM3.0_Boxed, symbol Connector:Screw_Terminal_01x01
- removed Q6, Q7: Q_PNP, symbol Device:Q_PNP
- removed Q8, Q9: Q_NPN, symbol Device:Q_NPN
- removed R14, R15, R16, R17: R_US, symbol Device:R_US
- removed RV2, RV3: R_Potentiometer_US, symbol Device:R_Potentiometer_US
- added C8, C9: 10nF, Capacitor_THT:C_Disc_D4.3mm_W1.9mm_P5.00mm, symbol Device:C
- added J0_12, J0_13, J0_14, J0_15: Screw_Terminal_01x03, TerminalBlock_Phoenix:TerminalBlock_Phoenix_PT-1,5-3-3.5-H_1x03_P3.50mm_Horizontal, symbol Connector:Screw_Terminal_01x03
- added Q10: IRG4PF50W, Package_TO_SOT_THT:TO-247-3_Vertical, symbol Transistor_IGBT:IRG4PF50W
- added R18, R19, R20, R21, R22, R23, R24, R25, R26, R27, R28, R29, R30, R31, R32, R33, R34: R_US, symbol Device:R_US
- added U17, U18: LM741, LM741_TH:LM471_TH, symbol Amplifier_Operational:LM741
- added U19: TLP250, Package_DIP:DIP-8_W7.62mm, symbol Driver_FET:TLP250
- added U20: L298HN, Package_TO_SOT_THT:TO-220-15_P2.54x2.54mm_StaggerOdd_Lead5.84mm_TabDown, symbol Driver_Motor:L298HN
- added U21: 4069, symbol 4xxx:4069
Connections:
- net GNDREF: now also C8.2, C9.2, J0_14.2 (Pin_2), J0_15.3 (Pin_3), Q10.3 (E), R19.2, R21.2, R23.2
- net at D3.2 (A): now also R30.2
- net at J0_3.2 (Pin_2): now also R34.1
- net at J0_10.3 (Pin_3): now also U20.13 (OUT3)
- net at J0_9.3 (Pin_3): now also U20.2 (OUT1)
- net at J0_9.1 (Pin_1): now also U20.3 (OUT2)
- net at J0_2.1 (Pin_1): now also R30.1
- net at J0_1.2 (Pin_2): now also R28.1
- net at J0_1.3 (Pin_3): now also R29.1
- net at U16.2 (-): now also R19.1, R20.2
- net at J0_3.1 (Pin_1): now also R33.1
- net at J0_2.2 (Pin_2): now also R31.1
- net at J0_2.3 (Pin_3): now also R32.1
- net at U15.2: now also U20.5 (IN1)
- net at U13.1: now also R18.2
- net at U15.1: now also U20.7 (IN2)
- net at D4.2 (A): now also R31.2
- net at D8.2 (A): now also R27.2
- net at D2.2 (A): now also R29.2
- net at D1.2 (A): now also R28.2
- net at J0_3.3 (Pin_3): now also R27.1
- net at D5.2 (A): now also R32.2
- net at D6.2 (A): now also R33.2
- net at J0_10.1 (Pin_1): now also U20.14 (OUT4)
- net at U16.6: now also J0_13.3 (Pin_3), R20.1
- net at D7.2 (A): now also R34.2
- net at U16.4 (V-): now also J0_12.3 (Pin_3), U17.4 (V-), U18.4 (V-)
- net at U16.7 (V+): now also J0_12.1 (Pin_1), U17.7 (V+), U18.7 (V+)
- new net: J0_13.2 (Pin_2), R22.1, U17.6
- new net: R21.1, R22.2, U17.2 (-)
- new net: J0_13.1 (Pin_1), R24.1, U18.6
- new net: R23.1, R24.2, U18.2 (-)
- new net: U20.10 (IN3), U21.2
- new net: U20.12 (IN4), U21.1
- new net: J0_14.1 (Pin_1), U19.8 (VCC)
- new net: J0_14.3 (Pin_3), U19.5 (VEE)
- new net: Q10.1 (G), R26.1
- new net: J0_15.1 (Pin_1), Q10.2 (C)
- new net: R26.2, U19.7 (VO)
- new net: C9.1, U18.3 (+)
- new net: C8.1, U17.3 (+)
- new net: R25.1, U19.2 (A)
Other:
- moved on the sheet: C7, J0_10, U16

Commit message: Actualización de PCB
Parts:
- removed J1-3, J1-4, J2-3, J2-4, J3-3, J3-4, J4-3, J4-4, J5-3, J5-4, J6-3, J6-4, J7-3, J7-4, J8-3, J8-4: Screw_Terminal_01x01, TerminalBlock_MetzConnect:TerminalBlock_MetzConnect_360271_1x01_Horizontal_ScrewM3.0_Boxed, symbol Connector:Screw_Terminal_01x01
- added J0_16: Screw_Terminal_01x03, TerminalBlock_Phoenix:TerminalBlock_Phoenix_PT-1,5-3-3.5-H_1x03_P3.50mm_Horizontal, symbol Connector:Screw_Terminal_01x03
- added R14, R15, R16, R17, R35, R36, R37, R38, R39, R40: R_US, Resistor_THT:R_Axial_DIN0411_L9.9mm_D3.6mm_P25.40mm_Horizontal, symbol Device:R_US
- D9: footprint (none) -> Diode_THT:Diode_Bridge_19.0x3.5x10.0mm_P5.0mm
- R1, R2, R3, R4, R5, R6, R7, R8: footprint Resistor_THT:R_Axial_DIN0207_L6.3mm_D2.5mm_P10.16mm_Horizontal -> Resistor_THT:R_Axial_DIN0411_L9.9mm_D3.6mm_P25.40mm_Horizontal
- R10, R11, R12, R13, R18, R19, R20, R21, R22, R23, R24, R25, R26, R27, R28, R29, R30, R31, R32, R33, R34, R9: footprint (none) -> Resistor_THT:R_Axial_DIN0411_L9.9mm_D3.6mm_P25.40mm_Horizontal
- RV1: footprint (none) -> Potentiometer_THT:Potentiometer_Bourns_3266W_Vertical
- U15, U21: footprint (none) -> Package_TO_SOT_SMD:SOT-353_SC-70-5
Connections:
- net at U9.2 (-), U9.6: now also R14.2
- net at U10.2 (-), U10.6: now also R15.2
- net at U20.1 (SENSE_A): now also R39.2
- net at U20.15 (SENSE_B): now also R40.2
- net at U20.4 (Vs): now also J0_16.2 (Pin_2)
- net at U20.8 (GND): now also J0_16.1 (Pin_1)
- net at U20.9 (Vss): now also J0_16.3 (Pin_3)
- net at U11.2 (-), U11.6: now also R16.2
- net at Q4.2 (B): now also R17.1
- net at Q1.1 (E): now also R38.1
- net at Q2.1 (E): now also R37.1
- net at Q2.2 (B): now also R15.1
- net at Q1.2 (B): now also R14.1
- net at Q4.1 (E): now also R35.1
- net at U12.2 (-), U12.6: now also R17.2
- net at Q3.1 (E): now also R36.1
- net at Q3.2 (B): now also R16.1
- removed net GNDREF: C3.2, C4.2, C5.2, C6.2, C7.2, C8.2, C9.2, J0_14.2 (Pin_2), J0_15.3 (Pin_3), J0_4.1 (Pin_1), J9_5.3 (Pin_3), Q10.3 (E), R19.2, R21.2, R23.2, U13.2
- new net: C3.2, C4.2, C5.2, C6.2, J0_4.1 (Pin_1), J9_5.3 (Pin_3), R35.2, R36.2, R37.2, R38.2
- new net: J0_14.2 (Pin_2), J0_15.3 (Pin_3), Q10.3 (E)
- new net: C7.2, C8.2, C9.2, R19.2, R21.2, R23.2
Other:
- moved on the sheet: 3V3a1, 3V3b1, 5Va1, 5Vb1, C1, C2, C3, C4, C5, C6, C7, C8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

Commit message: Versión preliminar del PCB
Parts:
- removed PX100, PX101, PX102, PX103, PX104, PX105, PX106, PX107, PX108, PX109, PX110, PX61, PX62, PX63, PX64, PX65, PX66, PX67, PX68, PX69, PX70, PX71, PX72, PX73, PX74, PX75, PX76, PX77, PX78, PX79, PX80, PX81, PX82, PX83, PX84, PX85, PX86, PX87, PX88, PX89, PX90, PX91, PX92, PX93, PX94, PX95, PX96, PX97, PX98, PX99: ~, Connector_Wire:SolderWire-0.75sqmm_1x01_D1.25mm_OD2.3mm, symbol Connector:Screw_Terminal_01x01
- added C10, C11: 100nF, Capacitor_THT:C_Disc_D4.3mm_W1.9mm_P5.00mm, symbol Device:C
Connections:
- net at R5.1, U5.3: now also PX50.1 (Pin_1)
- net at R3.1, U3.3: now also PX48.1 (Pin_1)
- net at PX123.1 (Pin_1): now also Q2.1 (E), R37.1
- net at C3.2, C4.2, C5.2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: now also J0_6.2 (Pin_2), J0_6.3 (Pin_3), PX120.1 (Pin_1)
- net at R12.1: now also J0_11.1 (Pin_1); no longer U14.4
- net at R12.2: now also PX54.1 (Pin_1), U14.4; no longer J0_11.3 (Pin_3)
- net at R39.1: now also J0_16.1 (Pin_1), PX111.1 (Pin_1), R40.1, U20.8 (GND), C10.1, C11.1
- net at PX59.1 (Pin_1): now also RV1.2
- net at PX55.1 (Pin_1): now also J0_11.3 (Pin_3), U14.3
- net at U20.12 (IN4), U21.1: now also PX112.1 (Pin_1)
- net at J0_16.2 (Pin_2), U20.4 (Vs): now also C11.2
- net at U15.1, U20.7 (IN2): now also PX113.1 (Pin_1)
- net at J0_16.3 (Pin_3), U20.9 (Vss): now also C10.2
- net at PX119.1 (Pin_1): now also C9.1, U18.3 (+)
- net at R8.1, U8.3: now also PX53.1 (Pin_1)
- net at J9_1.1 (Pin_1), R1.1, R1.2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: now also PX45.1 (Pin_1), PX46.1 (Pin_1)
- net at PX60.1 (Pin_1): now also RV1.3
- net at U16.7 (V+), U17.7 (V+), U18.7 (V+): now also J0_12.2 (Pin_2); no longer J0_12.1 (Pin_1)
- net at U16.4 (V-), U17.4 (V-), U18.4 (V-): now also J0_12.1 (Pin_1); no longer J0_12.3 (Pin_3)
- net at C7.1, U16.3 (+): now also PX117.1 (Pin_1)
- net at C7.2, C8.2, C9.2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: now also J0_12.3 (Pin_3), PX116.1 (Pin_1)
- net at PX58.1 (Pin_1): now also RV1.1
- net at PX118.1 (Pin_1): now also C8.1, U17.3 (+)
- net at PX52.1 (Pin_1): now also R7.1, U7.3
- net at U13.2: now also PX56.1 (Pin_1)
- net at R6.1, U6.3: now also PX51.1 (Pin_1)
- net at PX114.1 (Pin_1): now also U19.3 (C)
- net at R18.1: now also PX57.1 (Pin_1)
- net at PX122.1 (Pin_1): now also Q3.1 (E), R36.1
- net at Q4.1 (E), R35.1: now also PX121.1 (Pin_1)
- net at R2.1, U2.3: now also PX47.1 (Pin_1)
- net at R4.1, U4.3: now also PX49.1 (Pin_1)
- net at PX124.1 (Pin_1): now also Q1.1 (E), R38.1
- net at PX115.1 (Pin_1): now also R25.2
Other:
- moved on the sheet: C3, C4, C5, C6, C7, C8, C9, D1, D2, D3, D4, D5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

Commit message: Esquematico listo
Parts:
- removed D9: D_Bridge_+-AA, Diode_THT:Diode_Bridge_19.0x3.5x10.0mm_P5.0mm, symbol Device:D_Bridge_+-AA
- removed U15, U21: 4069, Package_TO_SOT_SMD:SOT-353_SC-70-5, symbol 4xxx:4069
- added D10: GBU8J, Diode_THT:Diode_Bridge_Vishay_GBU, symbol Diode_Bridge:GBU8J
- added PX61, PX62: ~, Connector_Wire:SolderWire-0.75sqmm_1x01_D1.25mm_OD2.3mm, symbol Connector:Screw_Terminal_01x01
- C1, C10, C11, C2, C3, C4, C5, C6, C7, C8, C9: footprint Capacitor_THT:C_Disc_D4.3mm_W1.9mm_P5.00mm -> Capacitor_THT:C_Disc_D5.1mm_W3.2mm_P5.00mm
- Q1, Q2, Q3, Q4: footprint Package_TO_SOT_THT:TO-39-3 -> Package_TO_SOT_THT:TO-92
Connections:
- net at R9.2: now also D10.3
- net at C10.1, C11.1, J0_16.1 (Pin_1)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: now also PX61.1 (Pin_1); no longer PX111.1 (Pin_1)
- net at U20.10 (IN3): now also PX111.1 (Pin_1)
- net at U20.12 (IN4): now also PX62.1 (Pin_1); no longer PX112.1 (Pin_1)
- net at U20.5 (IN1): now also PX113.1 (Pin_1)
- net at U20.7 (IN2): now also PX112.1 (Pin_1); no longer PX113.1 (Pin_1)
- net at C3.1, U12.3 (+): no longer J0_6.1 (Pin_1)
- net at C2.1: now also 3V3b1.1 (Pin_1), J4.18 (Pin_18)
- net at C2.2: now also GND3.1 (Pin_1), J4.20 (Pin_20)
- net at U14.2: now also D10.4 (-)
- net at R11.1: now also D10.1 (+)
- net at R10.2: now also D10.2
- net at GND1.1 (Pin_1), J1.1 (Pin_1): now also C1.2
- net at 3V3a1.1 (Pin_1), J1.3 (Pin_3): now also C1.1
Other:
- moved on the sheet: C1, C2, D1, D2, D3, D4, D5, D6, D7, D8, J0_1, J0_2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
