File: Hardware/PCB_HORNO/PCB_HORNO.kicad_sch (KiCad schematic)
At the start: 220 parts, among them J0_1 Screw_Terminal_01x03, J0_10 Screw_Terminal_01x03, J0_11 Screw_Terminal_01x03, J0_12 Screw_Terminal_01x03, J0_13 Screw_Terminal_01x03, J0_14 Screw_Terminal_01x03, J0_15 Screw_Terminal_01x03, J0_16 Screw_Terminal_01x03, J0_2 Screw_Terminal_01x03, J0_3 Screw_Terminal_01x03, J0_4 Screw_Terminal_01x03, J0_5 Screw_Terminal_01x03, J0_6 Screw_Terminal_01x03, J0_7 Screw_Terminal_01x03, J0_8 Screw_Terminal_01x03, J0_9 Screw_Terminal_01x03, J1 Screw_Terminal_01x20, J2 Screw_Terminal_01x20, J3 Screw_Terminal_01x20, J4 Screw_Terminal_01x20, J9_1 Screw_Terminal_01x03, J9_5 Screw_Terminal_01x03, Q1 2N2222, Q10 IRG4PF50W, Q2 2N2222, Q3 2N2222, Q4 2N2222, Q5 BTA16-800B, U1 TLP521-1, U10 LM741, U11 LM741, U12 LM741, U13 MOC3021M, U14 TLP521-1, U16 LM741, U17 LM741, U18 LM741, U19 TLP250, U2 TLP521-1, U20 L298HN, U3 TLP521-1, U4 TLP521-1, U5 TLP521-1, U6 TLP521-1, U7 TLP521-1, U8 TLP521-1, U9 LM741

Commit message: Reorganización del esquematico
Parts:
- removed C7: 10nF, Capacitor_THT:C_Disc_D5.1mm_W3.2mm_P5.00mm, symbol Device:C
- removed PX117: ~, Connector_Wire:SolderWire-0.75sqmm_1x01_D1.25mm_OD2.3mm, symbol Connector:Screw_Terminal_01x01
- removed U16: LM741, LM741_TH:LM471_TH, symbol Amplifier_Operational:LM741
- added J0_17, J0_18: Screw_Terminal_01x03, TerminalBlock_Phoenix:TerminalBlock_Phoenix_PT-1,5-3-3.5-H_1x03_P3.50mm_Horizontal, symbol Connector:Screw_Terminal_01x03
- added PX65, PX66: ~, Connector_Wire:SolderWire-0.75sqmm_1x01_D1.25mm_OD2.3mm, symbol Connector:Screw_Terminal_01x01
- added Q6: IRG4PF50W, Package_TO_SOT_THT:TO-247-3_Vertical, symbol Transistor_IGBT:IRG4PF50W
- added U15: TLP250, Package_DIP:DIP-8_W7.62mm, symbol Driver_FET:TLP250
Connections:
- net at R22.1, U17.6: now also J0_13.3 (Pin_3); no longer J0_13.2 (Pin_2)
- net at C8.2, C9.2, R21.2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: no longer J0_12.3 (Pin_3), PX116.1 (Pin_1), R19.2
- net at J0_6.1 (Pin_1): now also C3.1, U12.3 (+)
- net at R20.1: now also U15.2 (A); no longer J0_13.3 (Pin_3)
- net at R19.1: now also Q6.1 (G); no longer R20.2
- new net: J0_18.1 (Pin_1), Q6.2 (C)
- new net: J0_17.2 (Pin_2), J0_18.3 (Pin_3), Q6.3 (E)
- new net: J0_12.3 (Pin_3), PX116.1 (Pin_1)
- new net: PX65.1 (Pin_1), U15.3 (C)
- new net: J0_17.3 (Pin_3), U15.5 (VEE)
- new net: R19.2, U15.7 (VO)
- new net: J0_17.1 (Pin_1), U15.8 (VCC)
- new net: PX66.1 (Pin_1), R20.2
Other:
- company: (none) -> Digicontrol
- title: (none) -> Módulos para ESP32
- moved on the sheet: 3V3a1, 3V3b1, 5Va1, 5Vb1, C1, C10, C11, C2, C3, C4, C5, C6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

Commit message: Organizando elementos en PCB
Parts:
- added J0_19, J0_20: Screw_Terminal_01x03, TerminalBlock_Phoenix:TerminalBlock_Phoenix_PT-1,5-3-3.5-H_1x03_P3.50mm_Horizontal, symbol Connector:Screw_Terminal_01x03
- added PX63, PX64, PX67, PX68, PX69, PX70: ~, Connector_Wire:SolderWire-0.75sqmm_1x01_D1.25mm_OD2.3mm, symbol Connector:Screw_Terminal_01x01
- Q10, Q6: footprint Package_TO_SOT_THT:TO-247-3_Vertical -> Package_TO_SOT_THT:TO-264-3_Vertical
Connections:
- new net: J0_19.3 (Pin_3), PX68.1 (Pin_1)
- new net: J0_20.1 (Pin_1), PX67.1 (Pin_1)
- new net: J0_20.2 (Pin_2), PX64.1 (Pin_1)
- new net: J0_20.3 (Pin_3), PX63.1 (Pin_1)
- new net: J0_19.1 (Pin_1), PX70.1 (Pin_1)
- new net: J0_19.2 (Pin_2), PX69.1 (Pin_1)

Commit message: Actualización de esquematico
Parts:
- removed J0_11, J0_12, J0_15, J0_17, J0_4, J9_1, J9_5: Screw_Terminal_01x03, TerminalBlock_Phoenix:TerminalBlock_Phoenix_PT-1,5-3-3.5-H_1x03_P3.50mm_Horizontal, symbol Connector:Screw_Terminal_01x03
- removed PX114, PX115: ~, Connector_Wire:SolderWire-0.75sqmm_1x01_D1.25mm_OD2.3mm, symbol Connector:Screw_Terminal_01x01
- removed Q10: IRG4PF50W, Package_TO_SOT_THT:TO-264-3_Vertical, symbol Transistor_IGBT:IRG4PF50W
- added J0_21, J0_22, J0_23, J0_24, J0_25, J0_26: Screw_Terminal_01x03, TerminalBlock_Phoenix:TerminalBlock_Phoenix_PT-1,5-3-3.5-H_1x03_P3.50mm_Horizontal, symbol Connector:Screw_Terminal_01x03
- added K1, K2, K3, K4: Fujitsu_FTR-LYCA005x, Relay_THT:Relay_SPDT_Fujitsu_FTR-LYCA005x_FormC_Vertical, symbol Relay:Fujitsu_FTR-LYCA005x
- added PS1, PS2, PS3, PS4, PS5, PS6, PS7, PS8: MEE1S0315SC, Converter_DCDC:Converter_DCDC_Murata_MEE1SxxxxSC_THT, symbol Converter_DCDC:MEE1S0315SC
- added PX71, PX72, PX73, PX74, PX75, PX76, PX77, PX78, PX79, PX80, PX81, PX82, PX83, PX84, PX85, PX86, PX87, PX88, PX89, PX90: ~, Connector_Wire:SolderWire-0.75sqmm_1x01_D1.25mm_OD2.3mm, symbol Connector:Screw_Terminal_01x01
- added Q7: IRG4PF50W, Package_TO_SOT_THT:TO-264-3_Vertical, symbol Transistor_IGBT:IRG4PF50W
- added R41, R42, R43, R44, R45, R46, R47, R48, R49: R_US, Resistor_THT:R_Axial_DIN0411_L9.9mm_D3.6mm_P25.40mm_Horizontal, symbol Device:R_US
- added U16, U21, U22, U23: TLP521-1, Package_DIP:DIP-4_W7.62mm, symbol Isolator:Optocoupler_DC_PhotoNPN_AKEC
Connections:
- net at U1.4, U2.4, U3.4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: now also R49.2
- net at J0_18.3 (Pin_3), Q6.3 (E): now also PS1.3 (-Vout), PS2.4 (+Vout)
- net at PX68.1 (Pin_1): now also U16.2; no longer J0_19.3 (Pin_3)
- net at U10.4 (V-), U11.4 (V-), U12.4 (V-)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: now also U17.4 (V-), U18.4 (V-), PS7.3 (-Vout)
- net at U10.7 (V+), U11.7 (V+), U12.7 (V+)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: now also U17.7 (V+), U18.7 (V+), PS6.4 (+Vout)
- net at C3.2, C4.2, C5.2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: now also C8.2, C9.2, PX116.1 (Pin_1), R21.2, R23.2, PS6.3 (-Vout), PS7.4 (+Vout), PS8.3 (-Vout)
- net at R12.1: now also PS5.4 (+Vout), R49.1
- net at PX55.1 (Pin_1), U14.3: now also PX45.1 (Pin_1), PX46.1 (Pin_1), R1.1, R1.2, R2.2, R3.2, R4.2, R5.2, R6.2, R7.2, R8.2, U1.3, PS5.3 (-Vout)
- net at J0_14.1 (Pin_1): now also Q7.2 (C); no longer U19.8 (VCC)
- net at U19.5 (VEE): now also PS3.3 (-Vout); no longer J0_14.3 (Pin_3)
- net at J0_20.1 (Pin_1): now also U16.4; no longer PX67.1 (Pin_1)
- net at J0_20.2 (Pin_2): no longer PX64.1 (Pin_1)
- net at J0_20.3 (Pin_3): now also K1.A2, R42.1; no longer PX63.1 (Pin_1)
- net at Q1.3 (C), Q2.3 (C), Q3.3 (C)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: now also PS8.4 (+Vout)
- net at U15.5 (VEE): now also PS2.3 (-Vout)
- net at U15.8 (VCC): now also PS1.4 (+Vout)
- net at U19.3 (C): now also PX79.1 (Pin_1)
- net at R26.1: now also U19.2 (A)
- net at R26.2: now also PX80.1 (Pin_1); no longer U19.7 (VO)
- net at PX70.1 (Pin_1): now also U21.2; no longer J0_19.1 (Pin_1)
- net at PX69.1 (Pin_1): now also R41.2; no longer J0_19.2 (Pin_2)
- net at R25.2: now also U19.7 (VO)
- net at R25.1: now also Q7.1 (G); no longer U19.2 (A)
- new net: R44.1, U21.1
- new net: K2.A1, R43.2, U21.3
- new net: J0_22.1 (Pin_1), U21.4
- new net: PS3.2 (+Vin), PX77.1 (Pin_1)
- new net: PS1.1 (-Vin), PX76.1 (Pin_1)
- new net: PS1.2 (+Vin), PX75.1 (Pin_1)
- new net: PX71.1 (Pin_1), U23.2
- new net: PS6.1 (-Vin), PX83.1 (Pin_1)
- new net: PS6.2 (+Vin), PX84.1 (Pin_1)
- new net: J0_25.3 (Pin_3), K4.11
- new net: J0_25.1 (Pin_1), K4.12
- new net: J0_25.2 (Pin_2), K4.14
- new net: K4.A1, R47.2, U23.3
- new net: J0_26.3 (Pin_3), K4.A2, R47.1
- new net: J0_22.3 (Pin_3), K2.A2, R43.1
- new net: PS7.1 (-Vin), PX87.1 (Pin_1)
- new net: PS3.1 (-Vin), PX78.1 (Pin_1)
- new net: J0_14.3 (Pin_3), PS3.4 (+Vout), PS4.3 (-Vout), Q7.3 (E)
- new net: R41.1, U16.1
- new net: K1.A1, R42.2, U16.3
- new net: J0_21.1 (Pin_1), K2.12
- new net: J0_21.2 (Pin_2), K2.14
- new net: J0_21.3 (Pin_3), K2.11
- new net: R46.1, U22.1
- new net: PX64.1 (Pin_1), U22.2
- new net: K3.A1, R45.2, U22.3
- new net: J0_24.1 (Pin_1), U22.4
- new net: PX67.1 (Pin_1), R46.2
- new net: J0_19.3 (Pin_3), K1.11
- new net: J0_19.1 (Pin_1), K1.12
- new net: J0_19.2 (Pin_2), K1.14
- new net: PS8.1 (-Vin), PX89.1 (Pin_1)
- new net: PS8.2 (+Vin), PX90.1 (Pin_1)
- new net: PS4.1 (-Vin), PX82.1 (Pin_1)
- new net: PS4.2 (+Vin), PX81.1 (Pin_1)
- new net: PS4.4 (+Vout), U19.8 (VCC)
- new net: J0_23.3 (Pin_3), K3.11
- new net: J0_23.1 (Pin_1), K3.12
- new net: J0_23.2 (Pin_2), K3.14
- new net: J0_24.3 (Pin_3), K3.A2, R45.1
- new net: PX63.1 (Pin_1), R44.2
- new net: PX72.1 (Pin_1), R48.2
- new net: PS2.1 (-Vin), PX73.1 (Pin_1)
- new net: PS5.1 (-Vin), PX86.1 (Pin_1)
- new net: PS5.2 (+Vin), PX85.1 (Pin_1)
- new net: R48.1, U23.1
- new net: J0_26.1 (Pin_1), U23.4
- new net: PS7.2 (+Vin), PX88.1 (Pin_1)
- new net: PS2.2 (+Vin), PX74.1 (Pin_1)
Other:
- moved on the sheet: 3V3a1, 3V3b1, 5Va1, 5Vb1, C1, C10, C11, C2, C3, C4, C5, C6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

Commit message: Agregando diodos de rueda libre (flyback)
Parts:
- added D11, D12, D13, D14, D15, D16, D17, D9: 1N4007, Diode_THT:D_DO-41_SOD81_P10.16mm_Horizontal, symbol Diode:1N4007
Connections:
- net at K2.A1, R43.2, U21.3: now also D11.1 (K)
- net at J0_10.3 (Pin_3), U20.13 (OUT3): now also D14.1 (K), D15.2 (A)
- net at J0_10.1 (Pin_1), U20.14 (OUT4): now also D14.2 (A), D15.1 (K)
- net at J0_9.3 (Pin_3), U20.2 (OUT1): now also D16.1 (K), D17.2 (A)
- net at J0_9.1 (Pin_1), U20.3 (OUT2): now also D16.2 (A), D17.1 (K)
- net at K4.A1, R47.2, U23.3: now also D13.1 (K)
- net at J0_26.3 (Pin_3), K4.A2, R47.1: now also D13.2 (A)
- net at J0_22.3 (Pin_3), K2.A2, R43.1: now also D11.2 (A)
- net at J0_20.3 (Pin_3), K1.A2, R42.1: now also D9.2 (A)
- net at K1.A1, R42.2, U16.3: now also D9.1 (K)
- net at K3.A1, R45.2, U22.3: now also D12.1 (K)
- net at J0_24.3 (Pin_3), K3.A2, R45.1: now also D12.2 (A)
Other:
- moved on the sheet: C10, C11, C8, C9, J0_10, J0_13, J0_14, J0_16, J0_18, J0_19, J0_20, J0_21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

Commit message: Esquematico definitivo
Parts:
- removed D14, D15, D16, D17: 1N4007, Diode_THT:D_DO-41_SOD81_P10.16mm_Horizontal, symbol Diode:1N4007
- removed PX116, PX120, PX45, PX55, PX56, PX58, PX60, PX61, PX64, PX65, PX68, PX70, PX71, PX73, PX74, PX75, PX76, PX77, PX78, PX79, PX81, PX82, PX83, PX84, PX85, PX86, PX87, PX88, PX89, PX90: ~, Connector_Wire:SolderWire-0.75sqmm_1x01_D1.25mm_OD2.3mm, symbol Connector:Screw_Terminal_01x01
Connections:
- net at U16.2: now also C1.2, C10.1, C11.1, C3.2, C4.2, C5.2, C6.2, C8.2, C9.2, GND1.1 (Pin_1), J0_16.1 (Pin_1), J0_6.2 (Pin_2), J0_6.3 (Pin_3), J1.1 (Pin_1), PS1.1 (-Vin), PS2.1 (-Vin), PS3.1 (-Vin), PS4.1 (-Vin), PS5.1 (-Vin), PS5.3 (-Vout), PS6.1 (-Vin), PS6.3 (-Vout), PS7.1 (-Vin), PS7.4 (+Vout), PS8.1 (-Vin), PS8.3 (-Vout), PX46.1 (Pin_1), R1.1, R1.2, R2.2, R21.2, R23.2, R3.2, R35.2, R36.2, R37.2, R38.2, R39.1, R4.2, R40.1, R5.2, R6.2, R7.2, R8.2, RV1.1, U1.3, U13.2, U14.3, U15.3 (C), U19.3 (C), U20.8 (GND), U21.2, U22.2, U23.2
- net at PS3.2 (+Vin): now also 5Vb1.1 (Pin_1), J4.19 (Pin_19), PS1.2 (+Vin), PS2.2 (+Vin), PS4.2 (+Vin), PS6.2 (+Vin), PS7.2 (+Vin), PS8.2 (+Vin)
- net at RV1.3: now also 3V3a1.1 (Pin_1), C1.1, J1.3 (Pin_3), PS5.2 (+Vin)
Other:
- note removed: "Entradas/Salidas"

Commit message: Actualización de esquematico
Parts:
- added PX45, PX55: ~, Connector_Wire:SolderWire-0.75sqmm_1x01_D1.25mm_OD2.3mm, symbol Connector:Screw_Terminal_01x01
- R1, R12, R14, R15, R16, R17, R18, R19, R2, R20, R21, R22, R23, R24, R25, R26, R3, R35, R36, R37, R38, R4, R41, R44, R46, R48, R49, R5, R6, R7, R8: footprint Resistor_THT:R_Axial_DIN0411_L9.9mm_D3.6mm_P25.40mm_Horizontal -> Resistor_THT:R_Axial_DIN0207_L6.3mm_D2.5mm_P10.16mm_Horizontal
- R13, R27, R28, R29, R30, R31, R32, R33, R34, R39, R40, R42, R43, R45, R47: footprint Resistor_THT:R_Axial_DIN0411_L9.9mm_D3.6mm_P25.40mm_Horizontal -> Resistor_THT:R_Axial_DIN0309_L9.0mm_D3.2mm_P15.24mm_Horizontal
Connections:
- net at C1.2, C10.1, C11.1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: now also J0_13.2 (Pin_2)
- net at U20.11 (EnB): now also PX45.1 (Pin_1)
- net at U20.6 (EnA): now also PX55.1 (Pin_1)

Commit message: Ruteo de PCB
Connections:
- net at C1.2, C10.1, C11.1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: now also C2.2, GND3.1 (Pin_1), J4.20 (Pin_20); no longer PX46.1 (Pin_1), R1.1, U1.3
- net at 5Vb1.1 (Pin_1), J4.19 (Pin_19), PS1.2 (+Vin)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: no longer PS8.2 (+Vin)
- net at 3V3b1.1 (Pin_1), C2.1, J4.18 (Pin_18): now also PS8.2 (+Vin)
- new net: PX46.1 (Pin_1), R1.1, U1.3
Changed lines of the file:
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@@
 	)
 	(junction
+		(at 889 209.55)
+		(diameter 0)
+		(color 0 0 0 0)
+	)
+	(junction
 		(at 383.54 307.34)
 		(diameter 0)
@@
 	)
 	(junction
-		(at 195.58 121.92)
-		(diameter 0)
-		(color 0 0 0 0)
-	)
-	(junction
-		(at 842.01 104.14)
-		(diameter 0)
-		(color 0 0 0 0)
-	)
-	(junction
 		(at 961.39 204.47)
 		(diameter 0)
@@
 	)
 	(junction
+		(at 722.63 134.62)
+		(diameter 0)
+		(color 0 0 0 0)
+	)
+	(junction
 		(at 163.83 222.25)
 		(diameter 0)
@@
 	)
 	(junction
+		(at 727.71 100.33)
+		(diameter 0)
+		(color 0 0 0 0)
+	)
+	(junction
 		(at 419.1 105.41)
 		(diameter 0)
@@
 	(wire
 		(pts
-			(xy 868.68 104.14) (xy 842.01 104.14)
-		)
-		(stroke
-			(width 0)
-			(type default)
-			(color 255 6 0 1)
-		)
-	)
-	(wire
-		(pts
 			(xy 557.53 158.75) (xy 562.61 158.75)
 		)
@@
 	(wire
 		(pts
-			(xy 722.63 176.53) (xy 722.63 64.77)
+			(xy 722.63 176.53) (xy 722.63 134.62)
 		)
 		(stroke
 			(width 0)
 			(type default)
+			(color 255 6 0 1)
 		)
 	)
@@
 	(wire
 		(pts
+			(xy 722.63 134.62) (xy 722.63 64.77)
+		)
+		(stroke
+			(width 0)
+			(type default)
+			(color 255 6 0 1)
+		)
+	)
+	(wire
+		(pts
 			(xy 956.31 243.84) (xy 967.74 243.84)
 		)
@@
 	(wire
 		(pts
+			(xy 868.68 134.62) (xy 722.63 134.62)
+		)
+		(stroke
+			(width 0)
+			(type default)
+			(color 255 6 0 1)
+		)
+	)
+	(wire
+		(pts
 			(xy 106.68 152.4) (xy 97.79 152.4)
 		)
@@
 	(wire
 		(pts
-			(xy 727.71 176.53) (xy 727.71 59.69)
+			(xy 727.71 176.53) (xy 727.71 100.33)
 		)
 		(stroke
 			(width 0)
 			(type default)
+			(color 0 0 0 1)
 		)
 	)
@@
 	(wire
 		(pts
+			(xy 727.71 100.33) (xy 727.71 59.69)
+		)
+		(stroke
+			(width 0)
+			(type default)
+			(color 0 0 0 1)
+		)
+	)
+	(wire
+		(pts
 			(xy 715.01 176.53) (xy 715.01 72.39)
 		)
@@
 			(width 0)
 			(type default)
+			(color 255 6 0 1)
 		)
 	)
 	(wire
 		(pts
-			(xy 195.58 121.92) (xy 195.58 130.81)
+			(xy 195.58 105.41) (xy 195.58 130.81)
 		)
 		(stroke
@@
 			(width 0)
 			(type default)
+			(color 0 0 0 1)
 		)
 	)
@@
 			(width 0)
 			(type default)
+			(color 255 6 0 1)
 		)
 	)
@@
 	(wire
 		(pts
+			(xy 727.71 100.33) (xy 889 100.33)
+		)
+		(stroke
+			(width 0)
+			(type default)
+			(color 0 0 0 1)
+		)
+	)
+	(wire
+		(pts
 			(xy 1051.56 187.96) (xy 1098.55 187.96)
 		)
@@
 	(wire
 		(pts
-			(xy 868.68 104.14) (xy 868.68 236.22)
-		)
-		(stroke
-			(width 0)
-			(type default)
-			(color 255 6 0 1)
-		)
-	)
-	(wire
-		(pts
 			(xy 975.36 167.64) (xy 981.71 167.64)
 		)
@@
 	(wire
 		(pts
+			(xy 889 209.55) (xy 889 100.33)
+		)
+		(stroke
+			(width 0)
+			(type default)
+			(color 0 0 0 1)
+		)
+	)
+	(wire
+		(pts
 			(xy 622.3 322.58) (xy 622.3 363.22)
 		)
@@
 			(width 0)
 			(type default)
+			(color 0 0 0 1)
 		)
 	)
@@
 	(wire
 		(pts
-			(xy 171.45 121.92) (xy 195.58 121.92)
+			(xy 171.45 121.92) (xy 241.3 121.92)
 		)
 		(stroke
@@
 			(width 0)
 			(type default)
+			(color 255 6 0 1)
 		)
 	)
@@
 			(width 0)
 			(type default)
+			(color 255 6 0 1)
 		)
 	)
@@
 	(wire
 		(pts
+			(xy 868.68 134.62) (xy 868.68 236.22)
+		)
+		(stroke
+			(width 0)
+			(type default)
+			(color 255 6 0 1)
+		)
+	)
+	(wire
+		(pts
 			(xy 1027.43 165.1) (xy 1005.84 165.1)
 		)
@@
 	(wire
 		(pts
-			(xy 195.58 105.41) (xy 195.58 121.92)
-		)
-		(stroke
-			(width 0)
-			(type default)
-			(color 0 0 0 1)
-		)
-	)
-	(wire
-		(pts
 			(xy 514.35 176.53) (xy 514.35 115.57)
 		)
@@
 	(wire
 		(pts
-			(xy 195.58 121.92) (xy 241.3 121.92)
-		)
-		(stroke
-			(width 0)
-			(type default)
-		)
-	)
-	(wire
-		(pts
 			(xy 623.57 85.09) (xy 702.31 85.09)
 		)
@@
 			(width 0)
 			(type default)
+			(color 0 0 0 1)
 		)
 	)

Commit message: Ajustes a las interfaces digital y analogica
Parts:
- U10, U11, U12, U17, U18, U9: footprint LM741_TH:LM471_TH -> LM741_TH:LM741_TH
Changed lines of the file:
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@@
 			)
 		)
-		(property "Footprint" "LM741_TH:LM471_TH"
+		(property "Footprint" "LM741_TH:LM741_TH"
 			(at 996.95 166.37 0)
 			(effects
@@
 			)
 		)
-		(property "Footprint" "LM741_TH:LM471_TH"
+		(property "Footprint" "LM741_TH:LM741_TH"
 			(at 996.95 191.77 0)
 			(effects
@@
 			)
 		)
-		(property "Footprint" "LM741_TH:LM471_TH"
+		(property "Footprint" "LM741_TH:LM741_TH"
 			(at 819.15 288.29 0)
 			(effects
@@
 			)
 		)
-		(property "Footprint" "LM741_TH:LM471_TH"
+		(property "Footprint" "LM741_TH:LM741_TH"
 			(at 996.95 217.17 0)
 			(effects
@@
 			)
 		)
-		(property "Footprint" "LM741_TH:LM471_TH"
+		(property "Footprint" "LM741_TH:LM741_TH"
 			(at 819.15 328.93 0)
 			(effects
@@
 			)
 		)
-		(property "Footprint" "LM741_TH:LM471_TH"
+		(property "Footprint" "LM741_TH:LM741_TH"
 			(at 996.95 242.57 0)
 			(effects
