File: Hardware/PCB_HORNO/PCB_HORNO.kicad_sch (KiCad schematic)
At the start: 249 parts, among them J0_1 Screw_Terminal_01x03, J0_10 Screw_Terminal_01x03, J0_13 Screw_Terminal_01x03, J0_14 Screw_Terminal_01x03, J0_16 Screw_Terminal_01x03, J0_18 Screw_Terminal_01x03, J0_19 Screw_Terminal_01x03, J0_2 Screw_Terminal_01x03, J0_20 Screw_Terminal_01x03, J0_21 Screw_Terminal_01x03, J0_22 Screw_Terminal_01x03, J0_23 Screw_Terminal_01x03, J0_24 Screw_Terminal_01x03, J0_25 Screw_Terminal_01x03, J0_26 Screw_Terminal_01x03, J0_3 Screw_Terminal_01x03, J0_5 Screw_Terminal_01x03, J0_6 Screw_Terminal_01x03, J0_7 Screw_Terminal_01x03, J0_8 Screw_Terminal_01x03, J0_9 Screw_Terminal_01x03, J1 Screw_Terminal_01x20, J2 Screw_Terminal_01x20, J3 Screw_Terminal_01x20, J4 Screw_Terminal_01x20, K1 Fujitsu_FTR-LYCA005x, K2 Fujitsu_FTR-LYCA005x, K3 Fujitsu_FTR-LYCA005x, K4 Fujitsu_FTR-LYCA005x, Q1 2N2222, Q2 2N2222, Q3 2N2222, Q4 2N2222, Q5 BTA16-800B, Q6 IRG4PF50W, Q7 IRG4PF50W, U1 TLP521-1, U10 LM741, U11 LM741, U12 LM741, U13 MOC3021M, U14 TLP521-1, U15 TLP250, U16 TLP521-1, U17 LM741, U18 LM741, U19 TLP250, U2 TLP521-1, U20 L298HN, U21 TLP521-1, U22 TLP521-1, U23 TLP521-1, U3 TLP521-1, U4 TLP521-1, U5 TLP521-1, U6 TLP521-1, U7 TLP521-1, U8 TLP521-1, U9 LM741

Commit message: Listado de componentes para el PCB
Parts:
- J0_1, J0_10, J0_13, J0_14, J0_16, J0_18, J0_19, J0_2, J0_20, J0_21, J0_22, J0_23, J0_24, J0_25, J0_26, J0_3, J0_5, J0_6, J0_7, J0_8, J0_9: value Screw_Terminal_01x03 -> Terminales de tornillo espaciados en 3.5mm
- J1, J2, J3, J4: value Screw_Terminal_01x20 -> 20 Pin 2.54mm Header Male Breakable
- K1, K2, K3, K4: value Fujitsu_FTR-LYCA005x -> Fujitsu FTR-LYCA005x
- PS1, PS4, PS6, PS7: value MEE1S0315SC -> MEE1S0515SC
- PS2, PS3: value MEE1S0315SC -> MEE1S0505SC
- PS5: value MEE1S0315SC -> MEE1S0305SC
- PS8: value MEE1S0315SC -> MEE1S0303SC
- R1, R2, R3, R4, R5, R6, R7, R8: value 560 Ω 1/4 W -> 560Ω - 1/4 W
- R10, R11, R9: value R_US -> Depende de aplicación cruce por cero
- R12: value R_US -> 330Ω - 1/4 W
- R13: value R_US -> Depende de aplicación disparo con triac
- R14, R15, R16, R17: value R_US -> 7.5KΩ - 1/4 W
- R18, R20, R26, R41, R44, R46, R48: value R_US -> 270Ω - 1/4 W
- R19, R25: value R_US -> 10Ω - 1/4 W
- R21, R22, R23, R24: value R_US -> Depende de la aplicación salida analógica
- R27, R28, R29, R30, R31, R32, R33, R34, R49: value R_US -> 100 Ω - 1/4 W
- R35, R36, R37, R38: value R_US -> 39Ω - 1/4 W
- R39, R40: value R_US -> Depende de la aplicación puente H
- R42, R43, R45, R47: value R_US -> Depende de la tensión aplicada a la bobina del rele
- RV1: value R_Potentiometer_US -> 10KΩ Bourns 3266W
- U20: value L298HN -> L298HN Multiwatt15 H
Other:
- note added: "+15 voltios"
- note added: "-15 voltios"
- note added: "-5 voltios"
- note added: "0-10 voltios"
- note added: "3.3 voltios"
- note added: "5 voltios"
