File: Hardware/PCB_HORNO/PCB_HORNO.kicad_pcb (KiCad board)
At the start: 2 copper layers, 86 parts, among them J1 Screw_Terminal_01x20, J2 Screw_Terminal_01x20, J3 Screw_Terminal_01x20, J4 Screw_Terminal_01x20

Commit message: Integrando todas las interfaces
Parts:
- added D1: LED, LED_THT:LED_D4.0mm, F.Cu at (-6.57, 176.7)
- added D2: LED, LED_THT:LED_D4.0mm, F.Cu at (-6.57, 183.2)
- added D3: LED, LED_THT:LED_D4.0mm, F.Cu at (-0.10, 176.7)
- added D4: LED, LED_THT:LED_D4.0mm, F.Cu at (-0.10, 183.2)
- added D5: LED, LED_THT:LED_D4.0mm, F.Cu at (6.37, 176.7)
- added D6: LED, LED_THT:LED_D4.0mm, F.Cu at (6.37, 183.2)
- added D7: LED, LED_THT:LED_D4.0mm, F.Cu at (12.8, 176.7)
- added D8: LED, LED_THT:LED_D4.0mm, F.Cu at (12.8, 183.2)
- added J0_1: Screw_Terminal_01x03, TerminalBlock_Phoenix:TerminalBlock_Phoenix_PT-1,5-3-3.5-H_1x03_P3.50mm_Horizontal, F.Cu at (-58.2, 177.6)
- added J0_2: Screw_Terminal_01x03, TerminalBlock_Phoenix:TerminalBlock_Phoenix_PT-1,5-3-3.5-H_1x03_P3.50mm_Horizontal, F.Cu at (-58.2, 187.5)
- added J0_3: Screw_Terminal_01x03, TerminalBlock_Phoenix:TerminalBlock_Phoenix_PT-1,5-3-3.5-H_1x03_P3.50mm_Horizontal, F.Cu at (-58.2, 197.4)
- added J1-1: Screw_Terminal_01x01, TerminalBlock_MetzConnect:TerminalBlock_MetzConnect_360271_1x01_Horizontal_ScrewM3.0_Boxed, F.Cu at (-32.1, 220.0)
- added J1-2: Screw_Terminal_01x01, TerminalBlock_MetzConnect:TerminalBlock_MetzConnect_360271_1x01_Horizontal_ScrewM3.0_Boxed, F.Cu at (-32.1, 229.3)
- added J2-1: Screw_Terminal_01x01, TerminalBlock_MetzConnect:TerminalBlock_MetzConnect_360271_1x01_Horizontal_ScrewM3.0_Boxed, F.Cu at (-32.1, 238.7)
- added J2-2: Screw_Terminal_01x01, TerminalBlock_MetzConnect:TerminalBlock_MetzConnect_360271_1x01_Horizontal_ScrewM3.0_Boxed, F.Cu at (-32.1, 248.1)
- added J3-1: Screw_Terminal_01x01, TerminalBlock_MetzConnect:TerminalBlock_MetzConnect_360271_1x01_Horizontal_ScrewM3.0_Boxed, F.Cu at (-21.1, 220.0)
- added J3-2: Screw_Terminal_01x01, TerminalBlock_MetzConnect:TerminalBlock_MetzConnect_360271_1x01_Horizontal_ScrewM3.0_Boxed, F.Cu at (-21.1, 229.3)
- added J4-1: Screw_Terminal_01x01, TerminalBlock_MetzConnect:TerminalBlock_MetzConnect_360271_1x01_Horizontal_ScrewM3.0_Boxed, F.Cu at (-21.1, 238.7)
- added J4-2: Screw_Terminal_01x01, TerminalBlock_MetzConnect:TerminalBlock_MetzConnect_360271_1x01_Horizontal_ScrewM3.0_Boxed, F.Cu at (-21.1, 248.1)
- added J5-1: Screw_Terminal_01x01, TerminalBlock_MetzConnect:TerminalBlock_MetzConnect_360271_1x01_Horizontal_ScrewM3.0_Boxed, F.Cu at (-10.0, 220.0)
- added J5-2: Screw_Terminal_01x01, TerminalBlock_MetzConnect:TerminalBlock_MetzConnect_360271_1x01_Horizontal_ScrewM3.0_Boxed, F.Cu at (-10.0, 229.3)
- added J6-1: Screw_Terminal_01x01, TerminalBlock_MetzConnect:TerminalBlock_MetzConnect_360271_1x01_Horizontal_ScrewM3.0_Boxed, F.Cu at (-10.0, 238.7)
- added J6-2: Screw_Terminal_01x01, TerminalBlock_MetzConnect:TerminalBlock_MetzConnect_360271_1x01_Horizontal_ScrewM3.0_Boxed, F.Cu at (-10.0, 248.1)
- added J7-1: Screw_Terminal_01x01, TerminalBlock_MetzConnect:TerminalBlock_MetzConnect_360271_1x01_Horizontal_ScrewM3.0_Boxed, F.Cu at (1.04, 220.0)
- added J7-2: Screw_Terminal_01x01, TerminalBlock_MetzConnect:TerminalBlock_MetzConnect_360271_1x01_Horizontal_ScrewM3.0_Boxed, F.Cu at (1.04, 229.3)
- added J8-1: Screw_Terminal_01x01, TerminalBlock_MetzConnect:TerminalBlock_MetzConnect_360271_1x01_Horizontal_ScrewM3.0_Boxed, F.Cu at (1.04, 238.7)
- added J8-2: Screw_Terminal_01x01, TerminalBlock_MetzConnect:TerminalBlock_MetzConnect_360271_1x01_Horizontal_ScrewM3.0_Boxed, F.Cu at (1.04, 248.1)
- added J9_1: Screw_Terminal_01x03, TerminalBlock_Phoenix:TerminalBlock_Phoenix_PT-1,5-3-3.5-H_1x03_P3.50mm_Horizontal, F.Cu at (-58.2, 207.3)
- added J9_2: Screw_Terminal_01x03, TerminalBlock_Phoenix:TerminalBlock_Phoenix_PT-1,5-3-3.5-H_1x03_P3.50mm_Horizontal, F.Cu at (-58.2, 217.3)
- added J9_3: Screw_Terminal_01x03, TerminalBlock_Phoenix:TerminalBlock_Phoenix_PT-1,5-3-3.5-H_1x03_P3.50mm_Horizontal, F.Cu at (-58.2, 227.2)
- added J9_4: Screw_Terminal_01x03, TerminalBlock_Phoenix:TerminalBlock_Phoenix_PT-1,5-3-3.5-H_1x03_P3.50mm_Horizontal, F.Cu at (-58.2, 237.1)
- added PX45: ~, Connector_Wire:SolderWire-0.75sqmm_1x01_D1.25mm_OD2.3mm, F.Cu at (-35.2, 175.8)
- added PX46: ~, Connector_Wire:SolderWire-0.75sqmm_1x01_D1.25mm_OD2.3mm, F.Cu at (-35.2, 180.4)
- added PX47: ~, Connector_Wire:SolderWire-0.75sqmm_1x01_D1.25mm_OD2.3mm, F.Cu at (-35.2, 185.1)
- added PX48: ~, Connector_Wire:SolderWire-0.75sqmm_1x01_D1.25mm_OD2.3mm, F.Cu at (-35.2, 189.8)
- added PX49: ~, Connector_Wire:SolderWire-0.75sqmm_1x01_D1.25mm_OD2.3mm, F.Cu at (-35.2, 194.4)
- added PX50: ~, Connector_Wire:SolderWire-0.75sqmm_1x01_D1.25mm_OD2.3mm, F.Cu at (-35.2, 199.1)
- added PX51: ~, Connector_Wire:SolderWire-0.75sqmm_1x01_D1.25mm_OD2.3mm, F.Cu at (-35.2, 203.7)
- added PX52: ~, Connector_Wire:SolderWire-0.75sqmm_1x01_D1.25mm_OD2.3mm, F.Cu at (-35.2, 208.3)
- added PX53: ~, Connector_Wire:SolderWire-0.75sqmm_1x01_D1.25mm_OD2.3mm, F.Cu at (-35.2, 213.0)
- added PX54: ~, Connector_Wire:SolderWire-0.75sqmm_1x01_D1.25mm_OD2.3mm, F.Cu at (-30.4, 175.8)
- added PX55: ~, Connector_Wire:SolderWire-0.75sqmm_1x01_D1.25mm_OD2.3mm, F.Cu at (-30.4, 180.4)
- added PX56: ~, Connector_Wire:SolderWire-0.75sqmm_1x01_D1.25mm_OD2.3mm, F.Cu at (-30.4, 185.1)
- added PX57: ~, Connector_Wire:SolderWire-0.75sqmm_1x01_D1.25mm_OD2.3mm, F.Cu at (-30.4, 189.8)
- added PX58: ~, Connector_Wire:SolderWire-0.75sqmm_1x01_D1.25mm_OD2.3mm, F.Cu at (-30.4, 194.4)
- added PX59: ~, Connector_Wire:SolderWire-0.75sqmm_1x01_D1.25mm_OD2.3mm, F.Cu at (-30.4, 199.1)
- added PX60: ~, Connector_Wire:SolderWire-0.75sqmm_1x01_D1.25mm_OD2.3mm, F.Cu at (-30.4, 203.7)
- added PX61: ~, Connector_Wire:SolderWire-0.75sqmm_1x01_D1.25mm_OD2.3mm, F.Cu at (-30.4, 208.3)
- added PX62: ~, Connector_Wire:SolderWire-0.75sqmm_1x01_D1.25mm_OD2.3mm, F.Cu at (-30.4, 213.0)
- added PX63: ~, Connector_Wire:SolderWire-0.75sqmm_1x01_D1.25mm_OD2.3mm, F.Cu at (-25.5, 175.8)
- added PX64: ~, Connector_Wire:SolderWire-0.75sqmm_1x01_D1.25mm_OD2.3mm, F.Cu at (-25.5, 180.4)
- added PX65: ~, Connector_Wire:SolderWire-0.75sqmm_1x01_D1.25mm_OD2.3mm, F.Cu at (-25.5, 185.1)
- added PX66: ~, Connector_Wire:SolderWire-0.75sqmm_1x01_D1.25mm_OD2.3mm, F.Cu at (-25.5, 189.8)
- added PX67: ~, Connector_Wire:SolderWire-0.75sqmm_1x01_D1.25mm_OD2.3mm, F.Cu at (-25.5, 194.4)
- added PX68: ~, Connector_Wire:SolderWire-0.75sqmm_1x01_D1.25mm_OD2.3mm, F.Cu at (-25.5, 199.1)
- added PX69: ~, Connector_Wire:SolderWire-0.75sqmm_1x01_D1.25mm_OD2.3mm, F.Cu at (-25.5, 203.7)
- added PX70: ~, Connector_Wire:SolderWire-0.75sqmm_1x01_D1.25mm_OD2.3mm, F.Cu at (-25.5, 208.3)
- added PX71: ~, Connector_Wire:SolderWire-0.75sqmm_1x01_D1.25mm_OD2.3mm, F.Cu at (-25.5, 213.0)
- added PX72: ~, Connector_Wire:SolderWire-0.75sqmm_1x01_D1.25mm_OD2.3mm, F.Cu at (-20.7, 175.8)
- added PX73: ~, Connector_Wire:SolderWire-0.75sqmm_1x01_D1.25mm_OD2.3mm, F.Cu at (-20.7, 180.4)
- added PX74: ~, Connector_Wire:SolderWire-0.75sqmm_1x01_D1.25mm_OD2.3mm, F.Cu at (-20.7, 185.1)
- added PX75: ~, Connector_Wire:SolderWire-0.75sqmm_1x01_D1.25mm_OD2.3mm, F.Cu at (-20.7, 189.8)
- added PX76: ~, Connector_Wire:SolderWire-0.75sqmm_1x01_D1.25mm_OD2.3mm, F.Cu at (-20.7, 194.4)
- added PX77: ~, Connector_Wire:SolderWire-0.75sqmm_1x01_D1.25mm_OD2.3mm, F.Cu at (-20.7, 199.1)
- added PX78: ~, Connector_Wire:SolderWire-0.75sqmm_1x01_D1.25mm_OD2.3mm, F.Cu at (-20.7, 203.7)
- added PX79: ~, Connector_Wire:SolderWire-0.75sqmm_1x01_D1.25mm_OD2.3mm, F.Cu at (-20.7, 208.3)
- added PX80: ~, Connector_Wire:SolderWire-0.75sqmm_1x01_D1.25mm_OD2.3mm, F.Cu at (-20.7, 213.0)
- added PX81: ~, Connector_Wire:SolderWire-0.75sqmm_1x01_D1.25mm_OD2.3mm, F.Cu at (-15.8, 175.8)
- added PX82: ~, Connector_Wire:SolderWire-0.75sqmm_1x01_D1.25mm_OD2.3mm, F.Cu at (-15.8, 180.4)
- added PX83: ~, Connector_Wire:SolderWire-0.75sqmm_1x01_D1.25mm_OD2.3mm, F.Cu at (-15.8, 185.1)
- added PX84: ~, Connector_Wire:SolderWire-0.75sqmm_1x01_D1.25mm_OD2.3mm, F.Cu at (-15.8, 189.8)
- added PX85: ~, Connector_Wire:SolderWire-0.75sqmm_1x01_D1.25mm_OD2.3mm, F.Cu at (-15.8, 194.4)
- added PX86: ~, Connector_Wire:SolderWire-0.75sqmm_1x01_D1.25mm_OD2.3mm, F.Cu at (-15.8, 199.1)
- added PX87: ~, Connector_Wire:SolderWire-0.75sqmm_1x01_D1.25mm_OD2.3mm, F.Cu at (-15.8, 203.7)
- added PX88: ~, Connector_Wire:SolderWire-0.75sqmm_1x01_D1.25mm_OD2.3mm, F.Cu at (-15.8, 208.3)
- added PX89: ~, Connector_Wire:SolderWire-0.75sqmm_1x01_D1.25mm_OD2.3mm, F.Cu at (-15.8, 213.0)
- added PX90: ~, Connector_Wire:SolderWire-0.75sqmm_1x01_D1.25mm_OD2.3mm, F.Cu at (-11.0, 175.8)
- added PX91: ~, Connector_Wire:SolderWire-0.75sqmm_1x01_D1.25mm_OD2.3mm, F.Cu at (-11.0, 180.4)
- added PX92: ~, Connector_Wire:SolderWire-0.75sqmm_1x01_D1.25mm_OD2.3mm, F.Cu at (-11.0, 185.1)
- added R1: 560 Ω 1/4 W, Resistor_THT:R_Axial_DIN0207_L6.3mm_D2.5mm_P10.16mm_Horizontal, F.Cu at (8.14, 217.3)
- added R2: 560 Ω 1/4 W, Resistor_THT:R_Axial_DIN0207_L6.3mm_D2.5mm_P10.16mm_Horizontal, F.Cu at (8.14, 221.4)
- added R3: 560 Ω 1/4 W, Resistor_THT:R_Axial_DIN0207_L6.3mm_D2.5mm_P10.16mm_Horizontal, F.Cu at (8.14, 225.4)
- added R4: 560 Ω 1/4 W, Resistor_THT:R_Axial_DIN0207_L6.3mm_D2.5mm_P10.16mm_Horizontal, F.Cu at (8.14, 229.5)
- added R5: 560 Ω 1/4 W, Resistor_THT:R_Axial_DIN0207_L6.3mm_D2.5mm_P10.16mm_Horizontal, F.Cu at (8.14, 233.6)
- added R6: 560 Ω 1/4 W, Resistor_THT:R_Axial_DIN0207_L6.3mm_D2.5mm_P10.16mm_Horizontal, F.Cu at (8.14, 237.6)
- added R7: 560 Ω 1/4 W, Resistor_THT:R_Axial_DIN0207_L6.3mm_D2.5mm_P10.16mm_Horizontal, F.Cu at (8.14, 241.7)
- added R8: 560 Ω 1/4 W, Resistor_THT:R_Axial_DIN0207_L6.3mm_D2.5mm_P10.16mm_Horizontal, F.Cu at (8.14, 245.7)
- added U1: TLP521-1, Package_DIP:DIP-4_W7.62mm, F.Cu at (-46.8, 175.5)
- added U2: TLP521-1, Package_DIP:DIP-4_W7.62mm, F.Cu at (-46.8, 182.2)
- added U3: TLP521-1, Package_DIP:DIP-4_W7.62mm, F.Cu at (-46.8, 188.8)
- added U4: TLP521-1, Package_DIP:DIP-4_W7.62mm, F.Cu at (-46.8, 195.4)
- added U5: TLP521-1, Package_DIP:DIP-4_W7.62mm, F.Cu at (-46.8, 202.1)
- added U6: TLP521-1, Package_DIP:DIP-4_W7.62mm, F.Cu at (-46.8, 208.7)
- added U7: TLP521-1, Package_DIP:DIP-4_W7.62mm, F.Cu at (-46.8, 215.4)
- added U8: TLP521-1, Package_DIP:DIP-4_W7.62mm, F.Cu at (-46.8, 222.0)

Commit message: Reorganizando elementos
Parts:
- added C3: 10nF, Capacitor_THT:C_Disc_D4.3mm_W1.9mm_P5.00mm, F.Cu at (294.0, 168.3)
- added C4: 10nF, Capacitor_THT:C_Disc_D4.3mm_W1.9mm_P5.00mm, F.Cu at (294.0, 171.8)
- added C5: 10nF, Capacitor_THT:C_Disc_D4.3mm_W1.9mm_P5.00mm, F.Cu at (294.0, 175.2)
- added C6: 10nF, Capacitor_THT:C_Disc_D4.3mm_W1.9mm_P5.00mm, F.Cu at (294.0, 178.7)
- added J0_4: Screw_Terminal_01x03, TerminalBlock_Phoenix:TerminalBlock_Phoenix_PT-1,5-3-3.5-H_1x03_P3.50mm_Horizontal, F.Cu at (271.7, 133.3)
- added J0_5: Screw_Terminal_01x03, TerminalBlock_Phoenix:TerminalBlock_Phoenix_PT-1,5-3-3.5-H_1x03_P3.50mm_Horizontal, F.Cu at (271.7, 143.3)
- added J0_6: Screw_Terminal_01x03, TerminalBlock_Phoenix:TerminalBlock_Phoenix_PT-1,5-3-3.5-H_1x03_P3.50mm_Horizontal, F.Cu at (271.7, 153.2)
- added J1-3: Screw_Terminal_01x01, TerminalBlock_MetzConnect:TerminalBlock_MetzConnect_360271_1x01_Horizontal_ScrewM3.0_Boxed, F.Cu at (297.9, 133.9)
- added J1-4: Screw_Terminal_01x01, TerminalBlock_MetzConnect:TerminalBlock_MetzConnect_360271_1x01_Horizontal_ScrewM3.0_Boxed, F.Cu at (297.9, 143.2)
- added J2-3: Screw_Terminal_01x01, TerminalBlock_MetzConnect:TerminalBlock_MetzConnect_360271_1x01_Horizontal_ScrewM3.0_Boxed, F.Cu at (297.9, 152.6)
- added J2-4: Screw_Terminal_01x01, TerminalBlock_MetzConnect:TerminalBlock_MetzConnect_360271_1x01_Horizontal_ScrewM3.0_Boxed, F.Cu at (297.9, 161.9)
- added J3-3: Screw_Terminal_01x01, TerminalBlock_MetzConnect:TerminalBlock_MetzConnect_360271_1x01_Horizontal_ScrewM3.0_Boxed, F.Cu at (309.0, 133.9)
- added J3-4: Screw_Terminal_01x01, TerminalBlock_MetzConnect:TerminalBlock_MetzConnect_360271_1x01_Horizontal_ScrewM3.0_Boxed, F.Cu at (309.0, 143.2)
- added J4-3: Screw_Terminal_01x01, TerminalBlock_MetzConnect:TerminalBlock_MetzConnect_360271_1x01_Horizontal_ScrewM3.0_Boxed, F.Cu at (309.0, 152.6)
- added J4-4: Screw_Terminal_01x01, TerminalBlock_MetzConnect:TerminalBlock_MetzConnect_360271_1x01_Horizontal_ScrewM3.0_Boxed, F.Cu at (309.0, 161.9)
- added J5-3: Screw_Terminal_01x01, TerminalBlock_MetzConnect:TerminalBlock_MetzConnect_360271_1x01_Horizontal_ScrewM3.0_Boxed, F.Cu at (320.0, 133.9)
- added J5-4: Screw_Terminal_01x01, TerminalBlock_MetzConnect:TerminalBlock_MetzConnect_360271_1x01_Horizontal_ScrewM3.0_Boxed, F.Cu at (320.0, 143.2)
- added J6-3: Screw_Terminal_01x01, TerminalBlock_MetzConnect:TerminalBlock_MetzConnect_360271_1x01_Horizontal_ScrewM3.0_Boxed, F.Cu at (320.0, 152.6)
- added J6-4: Screw_Terminal_01x01, TerminalBlock_MetzConnect:TerminalBlock_MetzConnect_360271_1x01_Horizontal_ScrewM3.0_Boxed, F.Cu at (320.0, 161.9)
- added J7-3: Screw_Terminal_01x01, TerminalBlock_MetzConnect:TerminalBlock_MetzConnect_360271_1x01_Horizontal_ScrewM3.0_Boxed, F.Cu at (331.1, 133.9)
- added J7-4: Screw_Terminal_01x01, TerminalBlock_MetzConnect:TerminalBlock_MetzConnect_360271_1x01_Horizontal_ScrewM3.0_Boxed, F.Cu at (331.1, 143.2)
- added J8-3: Screw_Terminal_01x01, TerminalBlock_MetzConnect:TerminalBlock_MetzConnect_360271_1x01_Horizontal_ScrewM3.0_Boxed, F.Cu at (331.1, 152.6)
- added J8-4: Screw_Terminal_01x01, TerminalBlock_MetzConnect:TerminalBlock_MetzConnect_360271_1x01_Horizontal_ScrewM3.0_Boxed, F.Cu at (331.1, 161.9)
- added J9_5: Screw_Terminal_01x03, TerminalBlock_Phoenix:TerminalBlock_Phoenix_PT-1,5-3-3.5-H_1x03_P3.50mm_Horizontal, F.Cu at (271.7, 163.1)
- added J9_6: Screw_Terminal_01x03, TerminalBlock_Phoenix:TerminalBlock_Phoenix_PT-1,5-3-3.5-H_1x03_P3.50mm_Horizontal, F.Cu at (271.7, 173.0)
- added Q1: 2N2222, Package_TO_SOT_THT:TO-39-3, F.Cu at (284.4, 134.7)
- added Q2: 2N2222, Package_TO_SOT_THT:TO-39-3, F.Cu at (284.4, 145.6)
- added Q3: 2N2222, Package_TO_SOT_THT:TO-39-3, F.Cu at (284.4, 156.6)
- added Q4: 2N2222, Package_TO_SOT_THT:TO-39-3, F.Cu at (284.4, 167.5)
- added U10: LM741, LM741_TH:LM741_TH, F.Cu at (317.3, 172.2)
- added U11: LM741, LM741_TH:LM741_TH, F.Cu at (328.4, 172.2)
- added U12: LM741, LM741_TH:LM741_TH, F.Cu at (339.4, 172.2)
- added U9: LM741, LM741_TH:LM741_TH, F.Cu at (306.3, 172.2)

Commit message: Reorganizando elementos
Parts:
- removed J9_2, J9_3, J9_4, J9_6: Screw_Terminal_01x03, TerminalBlock_Phoenix:TerminalBlock_Phoenix_PT-1,5-3-3.5-H_1x03_P3.50mm_Horizontal
- added PX100: ~, Connector_Wire:SolderWire-0.75sqmm_1x01_D1.25mm_OD2.3mm, F.Cu at (109.3, 270.4)
- added PX101: ~, Connector_Wire:SolderWire-0.75sqmm_1x01_D1.25mm_OD2.3mm, F.Cu at (114.2, 237.8)
- added PX102: ~, Connector_Wire:SolderWire-0.75sqmm_1x01_D1.25mm_OD2.3mm, F.Cu at (114.2, 242.5)
- added PX103: ~, Connector_Wire:SolderWire-0.75sqmm_1x01_D1.25mm_OD2.3mm, F.Cu at (114.2, 247.2)
- added PX104: ~, Connector_Wire:SolderWire-0.75sqmm_1x01_D1.25mm_OD2.3mm, F.Cu at (114.2, 251.8)
- added PX105: ~, Connector_Wire:SolderWire-0.75sqmm_1x01_D1.25mm_OD2.3mm, F.Cu at (114.2, 256.4)
- added PX106: ~, Connector_Wire:SolderWire-0.75sqmm_1x01_D1.25mm_OD2.3mm, F.Cu at (114.2, 261.1)
- added PX107: ~, Connector_Wire:SolderWire-0.75sqmm_1x01_D1.25mm_OD2.3mm, F.Cu at (114.2, 265.8)
- added PX108: ~, Connector_Wire:SolderWire-0.75sqmm_1x01_D1.25mm_OD2.3mm, F.Cu at (114.2, 270.4)
- added PX109: ~, Connector_Wire:SolderWire-0.75sqmm_1x01_D1.25mm_OD2.3mm, F.Cu at (231.2, 238.2)
- added PX110: ~, Connector_Wire:SolderWire-0.75sqmm_1x01_D1.25mm_OD2.3mm, F.Cu at (231.2, 242.9)
- added PX111: ~, Connector_Wire:SolderWire-0.75sqmm_1x01_D1.25mm_OD2.3mm, F.Cu at (231.2, 247.6)
- added PX112: ~, Connector_Wire:SolderWire-0.75sqmm_1x01_D1.25mm_OD2.3mm, F.Cu at (231.2, 252.2)
- added PX113: ~, Connector_Wire:SolderWire-0.75sqmm_1x01_D1.25mm_OD2.3mm, F.Cu at (231.2, 256.9)
- added PX114: ~, Connector_Wire:SolderWire-0.75sqmm_1x01_D1.25mm_OD2.3mm, F.Cu at (231.2, 261.5)
- added PX115: ~, Connector_Wire:SolderWire-0.75sqmm_1x01_D1.25mm_OD2.3mm, F.Cu at (231.2, 266.1)
- added PX116: ~, Connector_Wire:SolderWire-0.75sqmm_1x01_D1.25mm_OD2.3mm, F.Cu at (231.2, 270.8)
- added PX117: ~, Connector_Wire:SolderWire-0.75sqmm_1x01_D1.25mm_OD2.3mm, F.Cu at (236.0, 238.2)
- added PX118: ~, Connector_Wire:SolderWire-0.75sqmm_1x01_D1.25mm_OD2.3mm, F.Cu at (236.0, 242.9)
- added PX119: ~, Connector_Wire:SolderWire-0.75sqmm_1x01_D1.25mm_OD2.3mm, F.Cu at (236.0, 247.6)
- added PX120: ~, Connector_Wire:SolderWire-0.75sqmm_1x01_D1.25mm_OD2.3mm, F.Cu at (236.0, 252.2)
- added PX121: ~, Connector_Wire:SolderWire-0.75sqmm_1x01_D1.25mm_OD2.3mm, F.Cu at (236.0, 256.9)
- added PX122: ~, Connector_Wire:SolderWire-0.75sqmm_1x01_D1.25mm_OD2.3mm, F.Cu at (236.0, 261.5)
- added PX123: ~, Connector_Wire:SolderWire-0.75sqmm_1x01_D1.25mm_OD2.3mm, F.Cu at (236.0, 266.1)
- added PX124: ~, Connector_Wire:SolderWire-0.75sqmm_1x01_D1.25mm_OD2.3mm, F.Cu at (236.0, 270.8)
- added PX93: ~, Connector_Wire:SolderWire-0.75sqmm_1x01_D1.25mm_OD2.3mm, F.Cu at (109.3, 237.8)
- added PX94: ~, Connector_Wire:SolderWire-0.75sqmm_1x01_D1.25mm_OD2.3mm, F.Cu at (109.3, 242.5)
- added PX95: ~, Connector_Wire:SolderWire-0.75sqmm_1x01_D1.25mm_OD2.3mm, F.Cu at (109.3, 247.2)
- added PX96: ~, Connector_Wire:SolderWire-0.75sqmm_1x01_D1.25mm_OD2.3mm, F.Cu at (109.3, 251.8)
- added PX97: ~, Connector_Wire:SolderWire-0.75sqmm_1x01_D1.25mm_OD2.3mm, F.Cu at (109.3, 256.4)
- added PX98: ~, Connector_Wire:SolderWire-0.75sqmm_1x01_D1.25mm_OD2.3mm, F.Cu at (109.3, 261.1)
- added PX99: ~, Connector_Wire:SolderWire-0.75sqmm_1x01_D1.25mm_OD2.3mm, F.Cu at (109.3, 265.8)
- U10, U11, U12, U9: footprint LM741_TH:LM741_TH -> LM741_TH:LM471_TH
- moved PX92 252.3 mm to (226.3, 270.8)
- moved PX90 252.3 mm to (226.3, 261.5)
- moved PX91 252.3 mm to (226.3, 266.1)
- moved PX81 250.7 mm to (221.4, 256.9)
- moved PX82 250.7 mm to (221.4, 261.5)
- moved PX83 250.7 mm to (221.4, 266.1)
- moved PX84 250.7 mm to (221.4, 270.8)
- moved PX73 249.3 mm to (216.6, 256.9)
- moved PX74 249.3 mm to (216.6, 261.5)
- moved PX76 249.3 mm to (216.6, 270.8)
- moved PX72 249.3 mm to (216.6, 252.2)
- moved PX75 249.3 mm to (216.6, 266.1)
- moved PX85 246.0 mm to (226.3, 238.2)
- moved PX86 246.0 mm to (226.3, 242.9)
- moved PX87 246.0 mm to (226.3, 247.6)
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Connections:
- J0_4 pad 1: Net-(J0_4-Pin_1) -> GNDREF
- J0_4 pad 3: GNDREF -> Net-(J0_4-Pin_3)
- J9_1 pad 2: Net-(J9_1-Pin_2) -> unconnected-(J9_1-Pin_2-Pad2)
- J9_5 pad 1: unconnected-(J9_5-Pin_1-Pad1) -> Net-(J9_5-Pin_1)
- J9_5 pad 3: unconnected-(J9_5-Pin_3-Pad3) -> GNDREF
- Q1 pad 3: Net-(Q1-C) -> Net-(J9_5-Pin_1)
- Q2 pad 3: Net-(Q1-C) -> Net-(J9_5-Pin_1)
- Q3 pad 3: Net-(Q1-C) -> Net-(J9_5-Pin_1)
- Q4 pad 3: Net-(Q1-C) -> Net-(J9_5-Pin_1)
- R1 pad 2: Net-(J9_1-Pin_2) -> Net-(J9_1-Pin_1)
- R2 pad 2: Net-(J9_1-Pin_2) -> Net-(J9_1-Pin_1)
- R3 pad 2: Net-(J9_1-Pin_2) -> Net-(J9_1-Pin_1)
- R4 pad 2: Net-(J9_1-Pin_2) -> Net-(J9_1-Pin_1)
- R5 pad 2: Net-(J9_1-Pin_2) -> Net-(J9_1-Pin_1)
- R6 pad 2: Net-(J9_1-Pin_2) -> Net-(J9_1-Pin_1)
- R7 pad 2: Net-(J9_1-Pin_2) -> Net-(J9_1-Pin_1)
- R8 pad 2: Net-(J9_1-Pin_2) -> Net-(J9_1-Pin_1)
- U10 pad 7: Net-(J0_4-Pin_1) -> Net-(J0_4-Pin_3)
- U11 pad 7: Net-(J0_4-Pin_1) -> Net-(J0_4-Pin_3)
- U12 pad 7: Net-(J0_4-Pin_1) -> Net-(J0_4-Pin_3)
- U9 pad 7: Net-(J0_4-Pin_1) -> Net-(J0_4-Pin_3)

Commit message: Actualización de PCB
Parts:
- removed J1-1, J1-2, J1-3, J1-4, J2-1, J2-2, J2-3, J2-4, J3-1, J3-2, J3-3, J3-4, J4-1, J4-2, J4-3, J4-4, J5-1, J5-2, J5-3, J5-4, J6-1, J6-2, J6-3, J6-4, J7-1, J7-2, J7-3, J7-4, J8-1, J8-2, J8-3, J8-4: Screw_Terminal_01x01, TerminalBlock_MetzConnect:TerminalBlock_MetzConnect_360271_1x01_Horizontal_ScrewM3.0_Boxed
- added C7: 10nF, Capacitor_THT:C_Disc_D4.3mm_W1.9mm_P5.00mm, F.Cu at (362.8, 368.1)
- added C8: 10nF, Capacitor_THT:C_Disc_D4.3mm_W1.9mm_P5.00mm, F.Cu at (362.8, 371.6)
- added C9: 10nF, Capacitor_THT:C_Disc_D4.3mm_W1.9mm_P5.00mm, F.Cu at (362.8, 375.0)
- added D9: D_Bridge_+-AA, Diode_THT:Diode_Bridge_19.0x3.5x10.0mm_P5.0mm, F.Cu at (-19.2, 356.4)
- added J0_10: Screw_Terminal_01x03, TerminalBlock_Phoenix:TerminalBlock_Phoenix_PT-1,5-3-3.5-H_1x03_P3.50mm_Horizontal, F.Cu at (152.6, 363.5)
- added J0_11: Screw_Terminal_01x03, TerminalBlock_Phoenix:TerminalBlock_Phoenix_PT-1,5-3-3.5-H_1x03_P3.50mm_Horizontal, F.Cu at (-42.6, 347.3)
- added J0_12: Screw_Terminal_01x03, TerminalBlock_Phoenix:TerminalBlock_Phoenix_PT-1,5-3-3.5-H_1x03_P3.50mm_Horizontal, F.Cu at (364.0, 350.7)
- added J0_13: Screw_Terminal_01x03, TerminalBlock_Phoenix:TerminalBlock_Phoenix_PT-1,5-3-3.5-H_1x03_P3.50mm_Horizontal, F.Cu at (364.0, 360.6)
- added J0_14: Screw_Terminal_01x03, TerminalBlock_Phoenix:TerminalBlock_Phoenix_PT-1,5-3-3.5-H_1x03_P3.50mm_Horizontal, F.Cu at (-42.6, 357.2)
- added J0_14: Screw_Terminal_01x03, TerminalBlock_Phoenix:TerminalBlock_Phoenix_PT-1,5-3-3.5-H_1x03_P3.50mm_Horizontal, F.Cu at (243.4, 362.3)
- added J0_15: Screw_Terminal_01x03, TerminalBlock_Phoenix:TerminalBlock_Phoenix_PT-1,5-3-3.5-H_1x03_P3.50mm_Horizontal, F.Cu at (243.4, 372.2)
- added J0_16: Screw_Terminal_01x03, TerminalBlock_Phoenix:TerminalBlock_Phoenix_PT-1,5-3-3.5-H_1x03_P3.50mm_Horizontal, F.Cu at (152.6, 373.4)
- added J0_7: Screw_Terminal_01x03, TerminalBlock_Phoenix:TerminalBlock_Phoenix_PT-1,5-3-3.5-H_1x03_P3.50mm_Horizontal, F.Cu at (49.5, 357.8)
- added J0_8: Screw_Terminal_01x03, TerminalBlock_Phoenix:TerminalBlock_Phoenix_PT-1,5-3-3.5-H_1x03_P3.50mm_Horizontal, F.Cu at (-42.6, 337.4)
- added J0_9: Screw_Terminal_01x03, TerminalBlock_Phoenix:TerminalBlock_Phoenix_PT-1,5-3-3.5-H_1x03_P3.50mm_Horizontal, F.Cu at (152.6, 353.6)
- added Q10: IRG4PF50W, Package_TO_SOT_THT:TO-247-3_Vertical, F.Cu at (256.5, 361.3)
- added Q5: BTA16-800B, Package_TO_SOT_THT:TO-220-3_Vertical, F.Cu at (50.0, 367.5)
- added R10: R_US, Resistor_THT:R_Axial_DIN0411_L9.9mm_D3.6mm_P25.40mm_Horizontal, F.Cu at (-30.9, 341.0)
- added R11: R_US, Resistor_THT:R_Axial_DIN0411_L9.9mm_D3.6mm_P25.40mm_Horizontal, F.Cu at (-30.9, 346.1)
- added R12: R_US, Resistor_THT:R_Axial_DIN0411_L9.9mm_D3.6mm_P25.40mm_Horizontal, F.Cu at (-30.9, 351.3)
- added R13: R_US, Resistor_THT:R_Axial_DIN0411_L9.9mm_D3.6mm_P25.40mm_Horizontal, F.Cu at (48.8, 345.9)
- added R14: R_US, Resistor_THT:R_Axial_DIN0411_L9.9mm_D3.6mm_P25.40mm_Horizontal, F.Cu at (470.4, 347.9)
- added R15: R_US, Resistor_THT:R_Axial_DIN0411_L9.9mm_D3.6mm_P25.40mm_Horizontal, F.Cu at (470.4, 353.1)
- added R16: R_US, Resistor_THT:R_Axial_DIN0411_L9.9mm_D3.6mm_P25.40mm_Horizontal, F.Cu at (470.4, 358.2)
- added R17: R_US, Resistor_THT:R_Axial_DIN0411_L9.9mm_D3.6mm_P25.40mm_Horizontal, F.Cu at (470.4, 363.4)
- added R18: R_US, Resistor_THT:R_Axial_DIN0411_L9.9mm_D3.6mm_P25.40mm_Horizontal, F.Cu at (48.8, 351.1)
- added R19: R_US, Resistor_THT:R_Axial_DIN0411_L9.9mm_D3.6mm_P25.40mm_Horizontal, F.Cu at (333.9, 349.1)
- added R20: R_US, Resistor_THT:R_Axial_DIN0411_L9.9mm_D3.6mm_P25.40mm_Horizontal, F.Cu at (333.9, 354.3)
- added R21: R_US, Resistor_THT:R_Axial_DIN0411_L9.9mm_D3.6mm_P25.40mm_Horizontal, F.Cu at (333.9, 359.4)
- added R22: R_US, Resistor_THT:R_Axial_DIN0411_L9.9mm_D3.6mm_P25.40mm_Horizontal, F.Cu at (333.9, 364.6)
- added R23: R_US, Resistor_THT:R_Axial_DIN0411_L9.9mm_D3.6mm_P25.40mm_Horizontal, F.Cu at (333.9, 369.7)
- added R24: R_US, Resistor_THT:R_Axial_DIN0411_L9.9mm_D3.6mm_P25.40mm_Horizontal, F.Cu at (333.9, 374.9)
- added R25: R_US, Resistor_THT:R_Axial_DIN0411_L9.9mm_D3.6mm_P25.40mm_Horizontal, F.Cu at (242.6, 350.4)
- added R26: R_US, Resistor_THT:R_Axial_DIN0411_L9.9mm_D3.6mm_P25.40mm_Horizontal, F.Cu at (242.6, 355.6)
- added R27: R_US, Resistor_THT:R_Axial_DIN0411_L9.9mm_D3.6mm_P25.40mm_Horizontal, F.Cu at (-177.5, 360.9)
- added R28: R_US, Resistor_THT:R_Axial_DIN0411_L9.9mm_D3.6mm_P25.40mm_Horizontal, F.Cu at (-177.5, 366.1)
- added R29: R_US, Resistor_THT:R_Axial_DIN0411_L9.9mm_D3.6mm_P25.40mm_Horizontal, F.Cu at (-177.5, 371.2)
- added R30: R_US, Resistor_THT:R_Axial_DIN0411_L9.9mm_D3.6mm_P25.40mm_Horizontal, F.Cu at (-177.5, 376.4)
- added R31: R_US, Resistor_THT:R_Axial_DIN0411_L9.9mm_D3.6mm_P25.40mm_Horizontal, F.Cu at (-177.5, 381.6)
- added R32: R_US, Resistor_THT:R_Axial_DIN0411_L9.9mm_D3.6mm_P25.40mm_Horizontal, F.Cu at (-177.5, 386.7)
- added R33: R_US, Resistor_THT:R_Axial_DIN0411_L9.9mm_D3.6mm_P25.40mm_Horizontal, F.Cu at (-177.5, 391.9)
- added R34: R_US, Resistor_THT:R_Axial_DIN0411_L9.9mm_D3.6mm_P25.40mm_Horizontal, F.Cu at (-177.5, 397.0)
- added R35: R_US, Resistor_THT:R_Axial_DIN0411_L9.9mm_D3.6mm_P25.40mm_Horizontal, F.Cu at (470.4, 368.5)
- added R36: R_US, Resistor_THT:R_Axial_DIN0411_L9.9mm_D3.6mm_P25.40mm_Horizontal, F.Cu at (470.4, 373.7)
- added R37: R_US, Resistor_THT:R_Axial_DIN0411_L9.9mm_D3.6mm_P25.40mm_Horizontal, F.Cu at (470.4, 378.8)
- added R38: R_US, Resistor_THT:R_Axial_DIN0411_L9.9mm_D3.6mm_P25.40mm_Horizontal, F.Cu at (470.4, 384.0)
- added R39: R_US, Resistor_THT:R_Axial_DIN0411_L9.9mm_D3.6mm_P25.40mm_Horizontal, F.Cu at (130.1, 341.7)
- added R40: R_US, Resistor_THT:R_Axial_DIN0411_L9.9mm_D3.6mm_P25.40mm_Horizontal, F.Cu at (130.1, 346.9)
- added R9: R_US, Resistor_THT:R_Axial_DIN0411_L9.9mm_D3.6mm_P25.40mm_Horizontal, F.Cu at (-30.9, 335.8)
- added RV1: R_Potentiometer_US, Potentiometer_THT:Potentiometer_Bourns_3266W_Vertical, F.Cu at (66.0, 364.6)
- added U13: MOC3021M, Package_DIP:DIP-6_W7.62mm, F.Cu at (60.9, 355.7)
- added U14: TLP521-1, Package_DIP:DIP-4_W7.62mm, F.Cu at (-31.3, 355.9)
- added U15: 4069, Package_TO_SOT_SMD:SOT-353_SC-70-5, F.Cu at (159.6, 341.1)
- added U16: LM741, LM741_TH:LM471_TH, F.Cu at (337.6, 341.0)
- added U17: LM741, LM741_TH:LM471_TH, F.Cu at (348.7, 341.0)
- added U18: LM741, LM741_TH:LM471_TH, F.Cu at (359.7, 341.0)
- added U19: TLP250, Package_DIP:DIP-8_W7.62mm, F.Cu at (254.8, 366.8)
- added U20: L298HN, Package_TO_SOT_THT:TO-220-15_P2.54x2.54mm_StaggerOdd_Lead5.84mm_TabDown, F.Cu at (130.1, 373.6)
- added U21: 4069, Package_TO_SOT_SMD:SOT-353_SC-70-5, F.Cu at (159.6, 345.1)
- R1, R2, R3, R4, R5, R6, R7, R8: footprint Resistor_THT:R_Axial_DIN0207_L6.3mm_D2.5mm_P10.16mm_Horizontal -> Resistor_THT:R_Axial_DIN0411_L9.9mm_D3.6mm_P25.40mm_Horizontal
- moved GND1 220.7 mm to (-24.2, 200.4), turned to 90 degrees
- moved GND3 219.1 mm to (314.2, 200.4), turned to -90 degrees
- moved 5Va1 215.0 mm to (-20.2, 200.4), turned to 90 degrees
- moved 5Vb1 213.5 mm to (310.2, 200.4), turned to -90 degrees
- moved 3V3a1 209.4 mm to (-16.2, 200.4), turned to 90 degrees
- moved 3V3b1 207.8 mm to (306.2, 200.4), turned to -90 degrees
- moved GND2 203.8 mm to (-12.2, 200.4), turned to 90 degrees
- moved P36 202.2 mm to (302.2, 200.4), turned to -90 degrees
- moved RX1 198.2 mm to (-8.20, 200.4), turned to 90 degrees
- moved P37 196.6 mm to (298.2, 200.4), turned to -90 degrees
- moved TX1 192.5 mm to (-4.20, 200.4), turned to 90 degrees
- moved P38 191.0 mm to (294.2, 200.4), turned to -90 degrees
- moved RST1 186.9 mm to (-0.20, 200.4), turned to 90 degrees
- moved P39 185.4 mm to (290.2, 200.4), turned to -90 degrees
- moved P0 181.3 mm to (3.80, 200.4), turned to 90 degrees
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Connections:
- net GNDREF renamed Net-(J0_4-Pin_1)
